File: pcb/console/console.kicad_sch (KiCad schematic)
At the start: 5 parts, among them J1 Micro_SD_Card, SW1 CherryMX, SW2 CherryMX, U1 RP2040-ZERO

Commit message: ordered prototype
Parts:
- added DPAD1: GBC, gameboy-color:GBC DPAD, symbol custom:DPAD
- J1: footprint Connector_Card:microSD_HC_Molex_47219-2001 -> Connector_Card:microSD_HC_Wuerth_693072010801
- renumbered SW1 to A1, SW2 to B1
Connections:
- net DOWN: now reaches U1.10 (GP9)
- net DOWN: now also DPAD1.5
- net LEFT: now reaches U1.11 (GP10)
- net LEFT: now also DPAD1.7
- net RIGHT: now reaches U1.12 (GP11)
- net RIGHT: now also DPAD1.3
- net SDA0: now reaches U1.13 (GP12)
- net SDA0: now also Brd1.4 (SDA)
- net SCL0: now reaches U1.14 (GP13)
- net SCL0: now also Brd1.3 (SCL)
- net CS: now reaches U1.2 (GP1)
- net CS: now also J1.2 (DAT3/CD)
- net +3.3V: now reaches U1.21 (3V3)
- net +3.3V: now also J1.4 (VDD)
- net GND: now reaches U1.22 (GND)
- net GND: now also A1.2, B1.2, Brd1.1 (GND), J1.6 (VSS), J1.9 (SHIELD), DPAD1.2, DPAD1.4, DPAD1.6, DPAD1.8
- net +5V: now reaches U1.23 (5V)
- net +5V: now also Brd1.2 (VCC)
- net SCLK: now reaches U1.3 (GP2)
- net SCLK: now also J1.5 (CLK)
- net MOSI: now reaches U1.4 (GP3)
- net MOSI: now also J1.3 (CMD)
- net MISO: now reaches U1.5 (GP4)
- net MISO: now also J1.7 (DAT0)
- net A: now reaches U1.7 (GP6)
- net A: now also A1.1
- net B: now reaches U1.8 (GP7)
- net B: now also B1.1
- net UP: now reaches U1.9 (GP8)
- net UP: now also DPAD1.1
